Commit message: renamed radar frame

File: urdf/radar.xacro (robot description, xacro)
@@ -3,7 +3,7 @@
     <joint name="radar_joint" type="fixed">
         <parent link="base_link"/>
-        <child link="radar_frame"/>
+        <child link="ti_mmwave_0"/>
         <origin xyz="0.2 0.05 0.08" rpy="0 0 0"/>
     </joint>
-    <link name="radar_frame"/>
+    <link name="ti_mmwave_0"/>
 </robot>
